File: Flatbox-rev8.kicad_pcb (KiCad board)
At the start: 2 copper layers, 272.6 x 171 mm, 78 parts, among them SW1 SW_Push, SW10 GPIO18, SW11 GPIO25, SW12 GPIO27, SW13 GPIO29, SW14 GPIO19, SW15 GPIO24, SW16 GPIO26, SW17 GPIO28, SW18 GPIO16, SW19 GPIO24, SW19 SW_Push, SW2 SW_Push, SW20 SW_Push, SW3 SW_Push, SW4 SW_Push, SW5 SW_Push, SW6 SW_Push, SW7 GPIO9, SW8 GPIO10, SW9 GPIO11, U1 RP2350_60QFN, U2 TLV73333PDBV, U3 W25Q128JVS, Y1 ABM8-272-T3

Commit message: final design inshallah
Parts:
- removed R9: 10k, Resistor_SMD:R_0402_1005Metric
- removed the REF** at (116.6, 92.8)
- removed the REF** at (97.6, 92.8)
- removed the REF** at (83.6, 43.9)
- added REF**: C_0402_1005Metric, PCM_JLCPCB:C_0402, F.Cu at (249.4, 146.0)
- added REF**: C_0603_1608Metric, PCM_JLCPCB:C_0603, F.Cu at (113.9, 73.3)
- added REF**: SOT-23-5, Package_TO_SOT_SMD:SOT-23-5, F.Cu at (153.7, 77.2)
- added REF**: C_0402_1005Metric, PCM_JLCPCB:C_0402, F.Cu at (100.5, 125.2)
- added REF**: LED_SK6812_EC15_1.5x1.5mm, LED_SMD:LED_SK6812_EC15_1.5x1.5mm, F.Cu at (106.9, 98.0)
- added REF**: C_0603_1608Metric, PCM_JLCPCB:C_0603, F.Cu at (113.9, 74.5)
- added REF**: LED_SK6812_EC15_1.5x1.5mm, LED_SMD:LED_SK6812_EC15_1.5x1.5mm, F.Cu at (253.5, 114.4)
- added REF**: LED_SK6812_EC15_1.5x1.5mm, LED_SMD:LED_SK6812_EC15_1.5x1.5mm, F.Cu at (197.9, 126.0)
- added REF**: LED_SK6812_EC15_1.5x1.5mm, LED_SMD:LED_SK6812_EC15_1.5x1.5mm, F.Cu at (98.9, 125.1)
- added REF**: LED_SK6812_EC15_1.5x1.5mm, LED_SMD:LED_SK6812_EC15_1.5x1.5mm, F.Cu at (218.9, 145.9)
- added REF**: LED_SK6812_EC15_1.5x1.5mm, LED_SMD:LED_SK6812_EC15_1.5x1.5mm, F.Cu at (224.2, 114.6)
- added REF**: C_0402_1005Metric, PCM_JLCPCB:C_0402, F.Cu at (184.6, 189.7)
- added REF**: C_0402_1005Metric, PCM_JLCPCB:C_0402, F.Cu at (225.8, 114.6)
- added REF**: C_0402_1005Metric, PCM_JLCPCB:C_0402, F.Cu at (217.6, 173.7)
- added REF**: LED_SK6812_EC15_1.5x1.5mm, LED_SMD:LED_SK6812_EC15_1.5x1.5mm, F.Cu at (216.0, 173.7)
- added REF**: C_0402_1005Metric, PCM_JLCPCB:C_0402, F.Cu at (108.6, 98.0)
- added REF**: R_0402_1005Metric, PCM_JLCPCB:R_0402, F.Cu at (152.7, 81.7)
- added REF**: LED_SK6812_EC15_1.5x1.5mm, LED_SMD:LED_SK6812_EC15_1.5x1.5mm, F.Cu at (199.4, 97.9)
- added REF**: LED_SK6812_EC15_1.5x1.5mm, LED_SMD:LED_SK6812_EC15_1.5x1.5mm, F.Cu at (182.9, 189.6)
- added REF**: C_0402_1005Metric, PCM_JLCPCB:C_0402, F.Cu at (220.6, 146.0)
- added REF**: C_0402_1005Metric, PCM_JLCPCB:C_0402, F.Cu at (255.1, 114.4)
- added REF**: C_0402_1005Metric, PCM_JLCPCB:C_0402, F.Cu at (127.1, 136.5)
- added REF**: LED_SK6812_EC15_1.5x1.5mm, LED_SMD:LED_SK6812_EC15_1.5x1.5mm, F.Cu at (69.8, 125.0)
- added REF**: LED_SK6812_EC15_1.5x1.5mm, LED_SMD:LED_SK6812_EC15_1.5x1.5mm, F.Cu at (280.7, 43.9)
- added REF**: C_0402_1005Metric, PCM_JLCPCB:C_0402, F.Cu at (144.6, 189.6)
- added REF**: LED_SK6812_EC15_1.5x1.5mm, LED_SMD:LED_SK6812_EC15_1.5x1.5mm, F.Cu at (192.3, 157.0)
- added REF**: LED_SK6812_EC15_1.5x1.5mm, LED_SMD:LED_SK6812_EC15_1.5x1.5mm, F.Cu at (247.8, 145.9)
- added REF**: C_0402_1005Metric, PCM_JLCPCB:C_0402, F.Cu at (201.1, 97.9)
- added REF**: LED_SK6812_EC15_1.5x1.5mm, LED_SMD:LED_SK6812_EC15_1.5x1.5mm, F.Cu at (125.5, 136.5)
- added REF**: C_0402_1005Metric, PCM_JLCPCB:C_0402, F.Cu at (278.6, 151.1)
- added REF**: LED_SK6812_EC15_1.5x1.5mm, LED_SMD:LED_SK6812_EC15_1.5x1.5mm, F.Cu at (277.0, 151.1)
- added REF**: LED_SK6812_EC15_1.5x1.5mm, LED_SMD:LED_SK6812_EC15_1.5x1.5mm, F.Cu at (286.7, 43.9)
- added REF**: LED_SK6812_EC15_1.5x1.5mm, LED_SMD:LED_SK6812_EC15_1.5x1.5mm, F.Cu at (143.0, 189.6)
- added REF**: C_0402_1005Metric, PCM_JLCPCB:C_0402, F.Cu at (156.3, 77.8)
- added REF**: C_0402_1005Metric, PCM_JLCPCB:C_0402, F.Cu at (284.1, 119.8)
- added REF**: C_0402_1005Metric, PCM_JLCPCB:C_0402, F.Cu at (194.0, 157.1)
- added REF**: LED_SK6812_EC15_1.5x1.5mm, LED_SMD:LED_SK6812_EC15_1.5x1.5mm, F.Cu at (282.4, 119.8)
- added REF**: C_0402_1005Metric, PCM_JLCPCB:C_0402, F.Cu at (199.6, 126.1)
- added REF**: LED_SK6812_EC15_1.5x1.5mm, LED_SMD:LED_SK6812_EC15_1.5x1.5mm, F.Cu at (283.7, 43.9)
- added REF**: C_0402_1005Metric, PCM_JLCPCB:C_0402, F.Cu at (71.4, 125.1)
- added REF**: LED_SK6812_EC15_1.5x1.5mm, LED_SMD:LED_SK6812_EC15_1.5x1.5mm, F.Cu at (289.7, 43.9)
- added U?: OLED-TH_L38.0-W12.0_HS91L02W2C01, EasyEDA_Lib:OLED-TH_L38.0-W12.0_HS91L02W2C01, F.Cu at (78.6, 43.9)
- SW1, SW3: renamed from SW8; footprint key-switches:SW_MX_Kailh_Choc_V1V2_HotSwap_Hybrid -> PCM_Switch_Keyboard_Hotswap_Kailh:SW_Hotswap_Kailh_Choc_V1V2
- SW10: renamed from SW16; footprint key-switches:SW_MX_Kailh_Choc_V1V2_HotSwap_Hybrid -> PCM_Switch_Keyboard_Hotswap_Kailh:SW_Hotswap_Kailh_Choc_V1V2
- SW11: renamed from SW17; footprint key-switches:SW_MX_Kailh_Choc_V1V2_HotSwap_Hybrid -> PCM_Switch_Keyboard_Hotswap_Kailh:SW_Hotswap_Kailh_Choc_V1V2
- SW12: renamed from SW10; footprint key-switches:SW_MX_Kailh_Choc_V1V2_HotSwap_Hybrid -> PCM_Switch_Keyboard_Hotswap_Kailh:SW_Hotswap_Kailh_Choc_V1V2
- SW13: renamed from SW11; footprint key-switches:SW_MX_Kailh_Choc_V1V2_HotSwap_Hybrid -> PCM_Switch_Keyboard_Hotswap_Kailh:SW_Hotswap_Kailh_Choc_V1V2
- SW14: renamed from SW12; footprint key-switches:SW_MX_Kailh_Choc_V1V2_HotSwap_Hybrid -> PCM_Switch_Keyboard_Hotswap_Kailh:SW_Hotswap_Kailh_Choc_V1V2
- SW15: renamed from SW13; footprint key-switches:SW_MX_Kailh_Choc_V1V2_HotSwap_Hybrid -> PCM_Switch_Keyboard_Hotswap_Kailh:SW_Hotswap_Kailh_Choc_V1V2
- SW16, SW7: renamed from SW19; footprint key-switches:SW_MX_Kailh_Choc_V1V2_HotSwap_Hybrid -> PCM_Switch_Keyboard_Hotswap_Kailh:SW_Hotswap_Kailh_Choc_V1V2
- SW19, SW20: footprint SW:C318884 -> Button_Switch_SMD:SW_SPST_EVQP2_ShortPushTravel_H2.1mm
- SW2: renamed from SW7; footprint key-switches:SW_MX_Kailh_Choc_V1V2_HotSwap_Hybrid -> PCM_Switch_Keyboard_Hotswap_Kailh:SW_Hotswap_Kailh_Choc_V1V2
- SW4: renamed from SW9; footprint key-switches:SW_MX_Kailh_Choc_V1V2_HotSwap_Hybrid -> PCM_Switch_Keyboard_Hotswap_Kailh:SW_Hotswap_Kailh_Choc_V1V2
- SW5, SW6: renamed from SW18; footprint key-switches:SW_MX_Kailh_Choc_V1V2_HotSwap_Hybrid -> PCM_Switch_Keyboard_Hotswap_Kailh:SW_Hotswap_Kailh_Choc_V1V2
- SW8: renamed from SW14; footprint key-switches:SW_MX_Kailh_Choc_V1V2_HotSwap_Hybrid -> PCM_Switch_Keyboard_Hotswap_Kailh:SW_Hotswap_Kailh_Choc_V1V2
- SW9: renamed from SW15; footprint key-switches:SW_MX_Kailh_Choc_V1V2_HotSwap_Hybrid -> PCM_Switch_Keyboard_Hotswap_Kailh:SW_Hotswap_Kailh_Choc_V1V2
- USB2: footprint Type-A:C2763302 -> Connector_USB:USB_A_TE_292303-7_Horizontal
- moved USB2 3.59 mm to (230.3, 62.4)
- moved C3 3.40 mm to (154.8, 58.0)
- moved C6 3.40 mm to (154.8, 59.0)
- moved R6 1.10 mm to (129.6, 71.9)
- moved Y1 1.03 mm to (143.6, 70.4)
- moved C16 1.03 mm to (142.2, 67.0)
- moved C17 1.03 mm to (145.2, 67.0)
- moved C10 0.86 mm to (142.0, 65.4)
- moved SW19 0.35 mm to (124.3, 67.0)
- moved C11 0.12 mm to (148.7, 53.0)
- moved R1 0.12 mm to (148.7, 51.1)
Connections:
- net /RUN renamed RESET
- SW1 pad 1: DOWN -> UP
- SW16 pad 1: CIRCLE -> LS
- SW5 pad 1: UP -> UP2
- SW6 pad 1: UP -> UP3
- SW7 pad 1: CIRCLE -> RS
- U1 pad 18: unconnected-(U1-GPIO14-Pad18) -> LS
- U1 pad 19: unconnected-(U1-GPIO15-Pad19) -> RS
- U1 pad 34: unconnected-(U1-GPIO22-Pad34) -> UP2
- U1 pad 35: unconnected-(U1-GPIO23-Pad35) -> UP3
- USB1 pad 3: unconnected-(USB1-SBU2-Pad3) -> (no net)
- USB1 pad 9: unconnected-(USB1-SBU1-Pad9) -> (no net)
Routing:
- net DOUT: track 0.00 -> 1048.4 mm, vias 0 -> 2
- net +5V: track 97.4 -> 995.4 mm, vias 2 -> 11
- net OPT6: track 35.4 -> 249.2 mm, vias 1 -> 2
- net OPT5: track 35.3 -> 238.0 mm, vias 1 -> 2
- net OPT4: track 35.8 -> 226.5 mm, vias 1 -> 2
- net RS: track 0.00 -> 186.6 mm, vias 0 -> 1
- net OPT3: track 31.1 -> 212.1 mm, vias 1 -> 2
- net OPT2: track 30.9 -> 200.7 mm, vias 1 -> 2
- net OPT1: track 30.8 -> 190.4 mm, vias 1 -> 2
- net UP3: track 0.00 -> 149.0 mm, vias 0 -> 3
- net UP2: track 0.00 -> 140.8 mm, vias 0 -> 3
- net SDA: track 0.00 -> 110.3 mm, vias 0 -> 2
- net SCL: track 0.00 -> 104.9 mm, vias 0 -> 2
- net LS: track 0.00 -> 78.0 mm, vias 0 -> 1
- net R1: track 188.9 -> 135.6 mm, vias 0 -> 1
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Other:
- outline, holes or cut-outs redrawn
- board text added: "GPIO13"
- board text added: "GPIO14"
- board text added: "GPIO15"
- board text added: "GPIO18"
- board text added: "GPIO19"
- board text added: "GPIO27"
- board text added: "GPIO29"
- board text added: "GPIO31"
- board text added: "GPIO34"
- board text added: "GPIO35"
- board text added: "GPIO36"
- board text added: "GPIO37"
- board text added: "GPIO40"
- board text added: "GPIO41"
- board text added: "GPIO42"
- board text added: "GPIO43"
- board text added: "rev1.4"
- board text removed: "rev1.2"
