File: Flatbox-rev8.kicad_pcb (KiCad board)
At the start: 2 copper layers, 272.6 x 171 mm, 116 parts, among them SW1 GPIO10, SW1 SW_Push, SW10 GPIO26, SW11 GPIO28, SW12 GPIO18, SW13 GPIO25, SW14 GPIO27, SW15 GPIO29, SW16 GPIO24, SW19 SW_Push, SW2 GPIO9, SW2 SW_Push, SW20 SW_Push, SW3 GPIO10, SW3 SW_Push, SW4 GPIO11, SW4 SW_Push, SW5 GPIO16, SW5 SW_Push, SW6 GPIO16, SW6 SW_Push, SW7 GPIO24, SW8 GPIO19, SW9 GPIO24, U1 RP2350_60QFN, U2 TLV73333PDBV, U3 W25Q128JVS, Y1 ABM8-272-T3

Commit message: Document PHBox design state and sync KiCad sources
Parts:
- R12, R13: renamed from REF**; value C_0603_1608Metric -> 4.7k; footprint PCM_JLCPCB:C_0603 -> PHBox:R_0603_Compact
- SW1: value GPIO10 -> GPIO16
- SW16: value GPIO24 -> GPIO14
- SW19, SW20: footprint Button_Switch_SMD:SW_SPST_EVQP2_ShortPushTravel_H2.1mm -> SW:C318884
- SW5: value GPIO16 -> GPIO22
- SW6: value GPIO16 -> GPIO23
- SW7: value GPIO24 -> GPIO15
- U5: renamed from U?; value OLED-TH_L38.0-W12.0_HS91L02W2C01 -> HS91L02W2C01
- USB2: footprint Connector_USB:USB_A_TE_292303-7_Horizontal -> Type-A:C2763302
- moved USB2 2.13 mm to (228.2, 62.4)
- renumbered SW1 to OPSW1, SW2 to OPSW2, SW3 to OPSW3, SW4 to OPSW4, SW5 to OPSW5, SW6 to OPSW6
Routing:
- net GND: track 76.3 -> 77.8 mm
- net +5V: track 995.4 -> 996.9 mm
- net HD-: track 76.8 -> 78.3 mm
- net HD+: track 76.7 -> 78.1 mm
Other:
- outline, holes or cut-outs redrawn

Commit message: Save validated PHBox design and document testing and manufacturing workflow
Parts:
- removed REF** (x20): LED_SK6812_EC15_1.5x1.5mm, LED_SMD:LED_SK6812_EC15_1.5x1.5mm
- added C36: 100n, lib:C_0402_1005Metric_small_pads, F.Cu at (280.7, 45.9)
- added C37: 100n, lib:C_0402_1005Metric_small_pads, F.Cu at (283.6, 45.9)
- added C38: 100n, lib:C_0402_1005Metric_small_pads, F.Cu at (286.6, 45.9)
- added C39: 100n, lib:C_0402_1005Metric_small_pads, F.Cu at (289.6, 45.9)
- added C41: 1u/10V/X7R, Capacitor_SMD:C_0603_1608Metric, B.Cu at (93.5, 42.4)
- added C42: 100n, Capacitor_SMD:C_0402_1005Metric, B.Cu at (216.6, 69.4)
- added C43: 100u/10V, PHBox:CP_KEMET_T520B_3528_21, B.Cu at (207.0, 62.4)
- added C44: 100n, Capacitor_SMD:C_0402_1005Metric, F.Cu at (221.4, 61.4)
- added D1: SK6805-EC15, PHBox_Repair:LED_SK6805_EC15_Optical, F.Cu at (106.9, 98.0)
- added D10: SK6805-EC15, PHBox_Repair:LED_SK6805_EC15_Optical, F.Cu at (247.8, 145.9)
- added D11: SK6805-EC15, PHBox_Repair:LED_SK6805_EC15_Optical, F.Cu at (277.0, 151.1)
- added D12: SK6805-EC15, PHBox_Repair:LED_SK6805_EC15_Optical, F.Cu at (197.9, 126.0)
- added D13: SK6805-EC15, PHBox_Repair:LED_SK6805_EC15_Optical, F.Cu at (224.2, 114.6)
- added D14: SK6805-EC15, PHBox_Repair:LED_SK6805_EC15_Optical, F.Cu at (253.5, 114.4)
- added D15: SK6805-EC15, PHBox_Repair:LED_SK6805_EC15_Optical, F.Cu at (282.4, 119.8)
- added D16: SK6805-EC15, PHBox_Repair:LED_SK6805_EC15_Optical, F.Cu at (199.4, 97.9)
- added D17: SK6805-EC15, PHBox_Repair:LED_SK6805_EC15_Optical, F.Cu at (280.7, 43.9)
- added D18: SK6805-EC15, PHBox_Repair:LED_SK6805_EC15_Optical, F.Cu at (283.7, 43.9)
- added D19: SK6805-EC15, PHBox_Repair:LED_SK6805_EC15_Optical, F.Cu at (286.7, 43.9)
- added D2: SK6805-EC15, PHBox_Repair:LED_SK6805_EC15_Optical, F.Cu at (69.8, 125.0)
- added D20: SK6805-EC15, PHBox_Repair:LED_SK6805_EC15_Optical, F.Cu at (289.7, 43.9)
- added D21: ESDA7P120-1U1M, Diode_SMD:ST_QFN-2L_1.6x1.0mm, F.Cu at (163.0, 47.0)
- added D3: SK6805-EC15, PHBox_Repair:LED_SK6805_EC15_Optical, F.Cu at (98.9, 125.1)
- added D4: SK6805-EC15, PHBox_Repair:LED_SK6805_EC15_Optical, F.Cu at (125.5, 136.5)
- added D5: SK6805-EC15, PHBox_Repair:LED_SK6805_EC15_Optical, F.Cu at (143.0, 189.6)
- added D6: SK6805-EC15, PHBox_Repair:LED_SK6805_EC15_Optical, F.Cu at (182.9, 189.6)
- added D7: SK6805-EC15, PHBox_Repair:LED_SK6805_EC15_Optical, F.Cu at (216.0, 173.7)
- added D8: SK6805-EC15, PHBox_Repair:LED_SK6805_EC15_Optical, F.Cu at (192.3, 157.0)
- added D9: SK6805-EC15, PHBox_Repair:LED_SK6805_EC15_Optical, F.Cu at (218.9, 145.9)
- added R15: 200k 1%, Resistor_SMD:R_0402_1005Metric, B.Cu at (211.5, 72.0)
- added R16: 10k, Resistor_SMD:R_0402_1005Metric, B.Cu at (220.0, 74.0)
- added R17: 10k, Resistor_SMD:R_0402_1005Metric, B.Cu at (211.5, 74.0)
- added R18: 100R, Resistor_SMD:R_0402_1005Metric, F.Cu at (98.2, 96.9)
- added R19: 100R, Resistor_SMD:R_0402_1005Metric, F.Cu at (78.2, 123.8)
- added R20: 100R, Resistor_SMD:R_0402_1005Metric, F.Cu at (107.2, 123.8)
- added R21: 100R, Resistor_SMD:R_0402_1005Metric, F.Cu at (133.8, 135.0)
- added R22: 100R, Resistor_SMD:R_0402_1005Metric, F.Cu at (151.4, 188.7)
- added R23: 100R, Resistor_SMD:R_0402_1005Metric, F.Cu at (174.4, 188.0)
- added R24: 100R, Resistor_SMD:R_0402_1005Metric, F.Cu at (207.4, 172.7)
- added R25: 100R, Resistor_SMD:R_0402_1005Metric, F.Cu at (200.8, 155.3)
- added R26: 100R, Resistor_SMD:R_0402_1005Metric, F.Cu at (227.4, 144.1)
- added R27: 100R, Resistor_SMD:R_0402_1005Metric, F.Cu at (256.6, 144.7)
- added R28: 100R, Resistor_SMD:R_0402_1005Metric, F.Cu at (268.6, 149.3)
- added R29: 100R, Resistor_SMD:R_0402_1005Metric, F.Cu at (206.2, 124.3)
- added R30: 100R, Resistor_SMD:R_0402_1005Metric, F.Cu at (233.0, 112.5)
- added R31: 100R, Resistor_SMD:R_0402_1005Metric, F.Cu at (261.8, 112.5)
- added R32: 100R, Resistor_SMD:R_0402_1005Metric, F.Cu at (274.0, 118.4)
- added R33: 100R, Resistor_SMD:R_0402_1005Metric, F.Cu at (190.8, 96.0)
- added U7: TPS2553DBVR, Package_TO_SOT_SMD:SOT-23-6, B.Cu at (216.3, 72.0)
- added U8: USBLC6-2SC6, Package_TO_SOT_SMD:SOT-23-6, B.Cu at (221.1, 62.4)
- C19: value 100u -> 100u/10V; footprint Capacitor_Tantalum_SMD:CP_EIA-3528-21_Kemet-B -> PHBox:CP_KEMET_T520B_3528_21
- C20, C21, C22, C23, C24, C25, C26, C27, C28, C29, C30, C31, C32, C33, C34, C35, C40: renamed from REF**; value C_0402_1005Metric -> 100n; footprint PCM_JLCPCB:C_0402 -> lib:C_0402_1005Metric_small_pads
- F1: value 500m -> 750mA hold
- R14: renamed from REF**; value R_0402_1005Metric -> 510R; footprint PCM_JLCPCB:R_0402 -> Resistor_SMD:R_0402_1005Metric
- SW1, SW10, SW11, SW12, SW13, SW14, SW15, SW16, SW2, SW3, SW4, SW5, SW6, SW7, SW8, SW9: footprint PCM_Switch_Keyboard_Hotswap_Kailh:SW_Hotswap_Kailh_Choc_V1V2 -> PHBox_Repair:SW_Hotswap_Kailh_Choc_V1V2_3D_Optical
- SW19, SW20: footprint SW:C318884 -> PHBox_Repair:SW_C318884_FabOnly
- U4: value ~ -> ECMF2-40A100N6; footprint ECMF02-4CMX8:ECMF02-4CMX8 -> PHBox:ECMF2-40A100N6
- U5: value HS91L02W2C01 -> WEA012864DWPP3N00003; footprint EasyEDA_Lib:OLED-TH_L38.0-W12.0_HS91L02W2C01 -> PHBox:OLED_WEA012864DWPP3N00003
- U6: renamed from REF**; value SOT-23-5 -> SN74LV1T34DBVR; footprint Package_TO_SOT_SMD:SOT-23-5 -> SOT-23-5:SOT-23-5
- moved U5 19.3 mm to (96.1, 52.0)
- moved C24 4.32 mm to (144.5, 194.0), turned to 0 degrees
- moved C32 3.93 mm to (226.0, 118.5), turned to 0 degrees
- moved C26 3.85 mm to (218.0, 177.5), turned to 0 degrees
- moved C33 3.62 mm to (255.1, 118.0), turned to 0 degrees
- moved C31 3.62 mm to (199.6, 129.7), turned to 0 degrees
- moved C22 3.62 mm to (100.5, 128.8), turned to 0 degrees
- moved C23 3.62 mm to (127.1, 140.2), turned to 0 degrees
- moved C27 3.62 mm to (194.0, 160.7), turned to 0 degrees
- moved C28 3.62 mm to (220.6, 149.6), turned to 0 degrees
- moved C29 3.62 mm to (249.4, 149.6), turned to 0 degrees
- moved C21 3.62 mm to (71.4, 128.7), turned to 0 degrees
- moved C35 3.62 mm to (201.1, 101.5), turned to 0 degrees
- moved C30 3.62 mm to (278.6, 154.8), turned to 0 degrees
- moved C25 3.62 mm to (184.6, 193.3), turned to 0 degrees
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Connections:
- net /FLASH_SS renamed /QSPI_SS
- net RESET renamed /RUN
- net RGB2 renamed /LED_BUFFER_Y
- C19 pad 1: +5V -> USB_HOST_5V
- R14 pad 2: DOUT -> /LED_DATA_IN
- U1 pad 10: unconnected-(U1-GPIO7-Pad10) -> USB_HOST_EN
- U1 pad 16: SCL -> SDA
- U1 pad 17: SDA -> SCL
- U1 pad 24: /SWCLK -> unconnected-(U1-SWCLK-Pad24)
- U1 pad 25: /SWD -> unconnected-(U1-SWD-Pad25)
- U1 pad 28: unconnected-(U1-GPIO17-Pad28) -> USB_HOST_FAULT_N
- U4 pad 1: +5V -> Net-(U4-D+_to_connector)
- U4 pad 3: Net-(USB1-DP1) -> GND
- U4 pad 4: unconnected-(U4-ID-Pad4) -> GND
- U4 pad 5: GND -> D-
- U5 pad 1: GND -> +3V3
- U5 pad 2: +5V -> GND
- U6 pad 1: (no net) -> unconnected-(U6-NC-Pad1)
- USB1 pad 3: (no net) -> unconnected-(USB1-SBU2-Pad3)
- USB1 pad 6: Net-(USB1-DP1) -> Net-(U4-D+_to_connector)
- USB1 pad 8: Net-(USB1-DP1) -> Net-(U4-D+_to_connector)
- USB1 pad 9: (no net) -> unconnected-(USB1-SBU1-Pad9)
- USB2 pad 1: +5V -> USB_HOST_5V
Routing:
- net DOUT: track 1048.4 -> 0.00 mm, vias 2 -> 0
- net +3V3: track 97.5 -> 241.5 mm, vias 2 -> 17
- net Net-(D16-DIN): track 0.00 -> 124.8 mm, vias 0 -> 2
- net Net-(D17-DIN): track 0.00 -> 122.6 mm, vias 0 -> 2
- net USB_HOST_EN: track 0.00 -> 122.2 mm, vias 0 -> 1
- net Net-(D12-DIN): track 0.00 -> 94.1 mm
- net USB_HOST_FAULT_N: track 0.00 -> 85.2 mm, vias 0 -> 3
- net /LED_DATA_IN: track 0.00 -> 75.8 mm, vias 0 -> 2
- net GND: track 77.8 -> 152.3 mm, vias 65 -> 177
- net Net-(D5-DIN): track 0.00 -> 64.9 mm
- net Net-(D2-DIN): track 0.00 -> 61.6 mm
- net +5V: track 996.9 -> 1057.5 mm, vias 11 -> 15
- net Net-(D7-DIN): track 0.00 -> 47.9 mm
- net USB_HOST_5V: track 0.00 -> 47.8 mm, vias 0 -> 4
- net SDA: track 110.3 -> 151.7 mm, vias 2 -> 5
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- added copper zone on B.Cu, net +1V1
- added copper zone on B.Cu, net +5V
- added copper zone on F.Cu, net /VREG_AVDD
- added copper zone on In1.Cu, net GND
- added copper zone on In2.Cu, net GND
- added copper zone on B.Cu, net USB_HOST_5V
- added copper zone on F.Cu, net USB_HOST_5V
Other:
- copper layers 2 -> 4
- rule pad_to_mask_clearance: 0.2 -> 0
